Commit message: 19200bps version

File: pandent_publisher/src/pandent_publisher/my_robot.urdf (robot description, URDF)
Before this commit: robot awesome-o, 19 links, 18 joints
Links:
- added link head; visual box size=0.06 0.06 0.04
Joints:
- added joint base_to_head: type revolute, parent base_link, child head, origin xyz=0.0 0 0.05 rpy=0 0 0, axis 0 0 1, limit lower=-3.14 upper=3.14 effort=1000.0 velocity=0.5
