Commit message: Hierarcy modified

File: pendant_publisher/urdf/pendant.urdf (robot description, URDF)
Before this commit: robot awesome-o, 19 links, 18 joints
Links:
- removed link base_link
- removed link left_forearm
- removed link left_shoulder
- removed link left_upper_arm
- removed link right_forearm
- removed link right_shoulder
- removed link right_upper_arm
- added link left_forearm_link; visual box size=0.03 0.04 0.09
- added link left_hand_link
- added link left_shoulder_link; visual box size=0.03 0.04 0.03
- added link left_upper_arm_link; visual box size=0.03 0.04 0.09
- added link right_forearm_link; visual box size=0.03 0.04 0.09
- added link right_hand_link
- added link right_shoulder_link; visual box size=0.03 0.04 0.03
- added link right_upper_arm_link; visual box size=0.03 0.04 0.09
- added link robot_head_link; visual box size=0.06 0.06 0.04
- added link torso_link; visual box size=0.11 0.05 0.12
Joints:
- removed joint base_to_left_shoulder
- removed joint base_to_right_shoulder
- added joint head: type fixed, parent torso_link, child robot_head_link, origin xyz=0.0 0 0.05 rpy=0 0 0
- added joint left_hand: type fixed, parent left_forearm_link, child left_hand_link, origin xyz=0.0 0 -0.09 rpy=0 0 0
- added joint left_shoulder: type revolute, parent torso_link, child left_shoulder_link, origin xyz=-0.07 0 0.03 rpy=1.5 0 0, axis -1 0 0, limit lower=-3.14 upper=3.14 effort=1000.0 velocity=0.5
- added joint right_hand: type fixed, parent right_forearm_link, child right_hand_link, origin xyz=0.0 0 -0.09 rpy=0 0 0
- added joint right_shoulder: type revolute, parent torso_link, child right_shoulder_link, origin xyz=0.07 0 0.03 rpy=1.5 0 0, axis 1 0 0, limit lower=-3.14 upper=3.14 effort=1000.0 velocity=0.5
- joint base_to_left_hip: parent base_link -> torso_link
- joint base_to_right_hip: parent base_link -> torso_link
- joint left_elbow: child left_forearm -> left_forearm_link; parent left_upper_arm -> left_upper_arm_link
- joint left_shoulder_to_upper: child left_upper_arm -> left_upper_arm_link; parent left_shoulder -> left_shoulder_link
- joint right_elbow: child right_forearm -> right_forearm_link; parent right_upper_arm -> right_upper_arm_link
- joint right_shoulder_to_upper: child right_upper_arm -> right_upper_arm_link; parent right_shoulder -> right_shoulder_link
